Commit message: Adjust visual model to base_link. base_link is in centre of rear axle
Signed-off-by: Lukasz Chojnacki <lukasz.chojnacki@robotec.ai>

File: cbus_vehicle_description/urdf/vehicle.xacro (robot description, xacro)
@@ -7,5 +7,5 @@
     <visual>
       <!-- <origin xyz="${vehicle_info['/**']['ros__parameters']['wheel_base']/2.0} 0 0" rpy="${pi/2.0} 0 ${pi}"/> -->
-      <origin xyz="-5.85 0 0" rpy="${pi/2.0} 0 ${pi}"/>
+      <origin xyz="-1.77 0 2.3" rpy="${pi/2.0} 0 ${pi}"/>
       <geometry>
         <mesh filename="package://cbus_vehicle_description/mesh/cbus.dae" scale="1 1 1"/>
